Commit message: fix launch files with fixed torso arg, added comments in bp

File: tiago/tiago_robot/tiago_description/urdf/torso/torso.urdf.xacro (robot description, xacro)
@@ -127,6 +127,6 @@
   <xacro:if value="$(arg fixed_torso)">
     <joint name="${name}_lift_joint" type="fixed">
-      <!-- Torso fixed height is set to half it's range -->
-      <origin rpy="0.0 0.0 0.0" xyz="0.0 0.0 0.772" />
+      <!-- Torso fixed height is set to half it's range (0.772)-->
+      <origin rpy="0.0 0.0 0.0" xyz="0.0 0.0 0.575" />
       <parent link="${name}_fixed_link" />
       <child link="${name}_lift_link" />

Commit message: minor changes in reuleaux - new simulation pkg wut_urdf_models (w/kitchen)

File: tiago/tiago_robot/tiago_description/urdf/torso/torso.urdf.xacro (robot description, xacro)
@@ -128,5 +128,5 @@
     <joint name="${name}_lift_joint" type="fixed">
       <!-- Torso fixed height is set to half it's range (0.772)-->
-      <origin rpy="0.0 0.0 0.0" xyz="0.0 0.0 0.575" />
+      <origin rpy="0.0 0.0 0.0" xyz="0.0 0.0 0.597" />
       <parent link="${name}_fixed_link" />
       <child link="${name}_lift_link" />
