Commit message: rename eut_urdf_models to sim_tiago_kitchen + bozza nodi nuovi e modifiche reuleaux

File: sim_tiago_kitchen/urdfs/sink.urdf.xacro (robot description, xacro)
@@ -15,11 +15,11 @@
             <origin xyz="0.0 0.0 0.0" rpy="1.5714 0.0 0.0"/>
             <geometry>
-                <mesh filename="package://eut_urdf_models/meshes/sink/kitchen_only_kitchen.obj" scale="100.0 100.0 100.0"/>
-            </geometry>
-        </visual>
-        <collision>
-            <origin xyz="0.0 0.0 0.0" rpy="1.5714 0.0 0.0"/>
-            <geometry>
-                <mesh filename="package://eut_urdf_models/meshes/sink/kitchen_only_kitchen.obj" scale="100.0 100.0 100.0"/>
+                <mesh filename="package://sim_tiago_kitchen/meshes/sink/kitchen_only_kitchen.obj" scale="100.0 100.0 100.0"/>
+            </geometry>
+        </visual>
+        <collision>
+            <origin xyz="0.0 0.0 0.0" rpy="1.5714 0.0 0.0"/>
+            <geometry>
+                <mesh filename="package://sim_tiago_kitchen/meshes/sink/kitchen_only_kitchen.obj" scale="100.0 100.0 100.0"/>
             </geometry>
         </collision>
@@ -42,11 +42,11 @@
             <origin xyz="0.0 0.0 0.0" rpy="1.5714 0.0 0.0"/>
             <geometry>
-                <mesh filename="package://eut_urdf_models/meshes/sink/kitchen_only_cajon_1.obj"/>
-            </geometry>
-        </visual>
-        <collision>
-            <origin xyz="0.0 0.0 0.0" rpy="1.5714 0.0 0.0"/>
-            <geometry>
-                <mesh filename="package://eut_urdf_models/meshes/sink/kitchen_only_cajon_1.obj"/>
+                <mesh filename="package://sim_tiago_kitchen/meshes/sink/kitchen_only_cajon_1.obj"/>
+            </geometry>
+        </visual>
+        <collision>
+            <origin xyz="0.0 0.0 0.0" rpy="1.5714 0.0 0.0"/>
+            <geometry>
+                <mesh filename="package://sim_tiago_kitchen/meshes/sink/kitchen_only_cajon_1.obj"/>
             </geometry>
         </collision>
@@ -68,11 +68,11 @@
             <origin xyz="0.0 0.0 0.0" rpy="1.5714 0.0 0.0"/>
             <geometry>
-                <mesh filename="package://eut_urdf_models/meshes/sink/kitchen_only_cajon_2.obj"/>
-            </geometry>
-        </visual>
-        <collision>
-            <origin xyz="0.0 0.0 0.0" rpy="1.5714 0.0 0.0"/>
-            <geometry>
-                <mesh filename="package://eut_urdf_models/meshes/sink/kitchen_only_cajon_2.obj"/>
+                <mesh filename="package://sim_tiago_kitchen/meshes/sink/kitchen_only_cajon_2.obj"/>
+            </geometry>
+        </visual>
+        <collision>
+            <origin xyz="0.0 0.0 0.0" rpy="1.5714 0.0 0.0"/>
+            <geometry>
+                <mesh filename="package://sim_tiago_kitchen/meshes/sink/kitchen_only_cajon_2.obj"/>
             </geometry>
         </collision>
@@ -95,11 +95,11 @@
             <origin xyz="0.0 0.0 0.0" rpy="1.5714 0.0 0.0"/>
             <geometry>
-                <mesh filename="package://eut_urdf_models/meshes/sink/kitchen_only_cajon_grande.obj"/>
-            </geometry>
-        </visual>
-        <collision>
-            <origin xyz="0.0 0.0 0.0" rpy="1.5714 0.0 0.0"/>
-            <geometry>
-                <mesh filename="package://eut_urdf_models/meshes/sink/kitchen_only_cajon_grande.obj"/>
+                <mesh filename="package://sim_tiago_kitchen/meshes/sink/kitchen_only_cajon_grande.obj"/>
+            </geometry>
+        </visual>
+        <collision>
+            <origin xyz="0.0 0.0 0.0" rpy="1.5714 0.0 0.0"/>
+            <geometry>
+                <mesh filename="package://sim_tiago_kitchen/meshes/sink/kitchen_only_cajon_grande.obj"/>
             </geometry>
         </collision>
@@ -122,5 +122,5 @@
             <origin xyz="0.3 0.0 0.0" rpy="1.5714 0.0 0.0"/>
             <geometry>
-                <mesh filename="package://eut_urdf_models/meshes/sink/kitchen_only_armario_lavamanos.obj"/>
+                <mesh filename="package://sim_tiago_kitchen/meshes/sink/kitchen_only_armario_lavamanos.obj"/>
             </geometry>
         </visual>
@@ -128,5 +128,5 @@
             <origin xyz="0.3 0.0 0.0" rpy="1.5714 0.0 0.0"/>
             <geometry>
-                <mesh filename="package://eut_urdf_models/meshes/sink/kitchen_only_armario_lavamanos.obj"/>
+                <mesh filename="package://sim_tiago_kitchen/meshes/sink/kitchen_only_armario_lavamanos.obj"/>
             </geometry>
         </collision>
@@ -149,5 +149,5 @@
             <origin xyz="0.0 0.0 0.254" rpy="1.5714 0.0 0.0"/>
             <geometry>
-                <mesh filename="package://eut_urdf_models/meshes/sink/kitchen_only_puerta_lavavajillas.obj"/>
+                <mesh filename="package://sim_tiago_kitchen/meshes/sink/kitchen_only_puerta_lavavajillas.obj"/>
             </geometry>
         </visual>
@@ -155,5 +155,5 @@
             <origin xyz="0.0 0.0 0.254" rpy="1.5714 0.0 0.0"/>
             <geometry>
-                <mesh filename="package://eut_urdf_models/meshes/sink/kitchen_only_puerta_lavavajillas.obj"/>
+                <mesh filename="package://sim_tiago_kitchen/meshes/sink/kitchen_only_puerta_lavavajillas.obj"/>
             </geometry>
         </collision>
@@ -175,11 +175,11 @@
             <origin xyz="-0.0 0.0 0.0" rpy="1.5714 0.0 0.0"/>
             <geometry>
-                <mesh filename="package://eut_urdf_models/meshes/sink/kitchen_only_lavadora.obj"/>
-            </geometry>
-        </visual>
-        <collision>
-            <origin xyz="0.0 0.0 0.0" rpy="1.5714 0.0 0.0"/>
-            <geometry>
-                <mesh filename="package://eut_urdf_models/meshes/sink/kitchen_only_lavadora.obj"/>
+                <mesh filename="package://sim_tiago_kitchen/meshes/sink/kitchen_only_lavadora.obj"/>
+            </geometry>
+        </visual>
+        <collision>
+            <origin xyz="0.0 0.0 0.0" rpy="1.5714 0.0 0.0"/>
+            <geometry>
+                <mesh filename="package://sim_tiago_kitchen/meshes/sink/kitchen_only_lavadora.obj"/>
             </geometry>
         </collision>
@@ -202,11 +202,11 @@
             <origin xyz="0.0 0.0 0.0" rpy="1.5714 0.0 0.0"/>
             <geometry>
-                <mesh filename="package://eut_urdf_models/meshes/sink/kitchen_only_parte_de_abajo_lavavajillas.obj"/>
-            </geometry>
-        </visual>
-        <collision>
-            <origin xyz="0.0 0.0 0.0" rpy="1.5714 0.0 0.0"/>
-            <geometry>
-                <mesh filename="package://eut_urdf_models/meshes/sink/kitchen_only_parte_de_abajo_lavavajillas.obj"/>
+                <mesh filename="package://sim_tiago_kitchen/meshes/sink/kitchen_only_parte_de_abajo_lavavajillas.obj"/>
+            </geometry>
+        </visual>
+        <collision>
+            <origin xyz="0.0 0.0 0.0" rpy="1.5714 0.0 0.0"/>
+            <geometry>
+                <mesh filename="package://sim_tiago_kitchen/meshes/sink/kitchen_only_parte_de_abajo_lavavajillas.obj"/>
             </geometry>
         </collision>
@@ -229,11 +229,11 @@
             <origin xyz="0.0 0.0 0.0" rpy="1.5714 0.0 0.0"/>
             <geometry>
-                <mesh filename="package://eut_urdf_models/meshes/sink/kitchen_only_parte_de_arriba_lavavajillas.obj"/>
-            </geometry>
-        </visual>
-        <collision>
-            <origin xyz="0.0 0.0 0.0" rpy="1.5714 0.0 0.0"/>
-            <geometry>
-                <mesh filename="package://eut_urdf_models/meshes/sink/kitchen_only_parte_de_arriba_lavavajillas.obj"/>
+                <mesh filename="package://sim_tiago_kitchen/meshes/sink/kitchen_only_parte_de_arriba_lavavajillas.obj"/>
+            </geometry>
+        </visual>
+        <collision>
+            <origin xyz="0.0 0.0 0.0" rpy="1.5714 0.0 0.0"/>
+            <geometry>
+                <mesh filename="package://sim_tiago_kitchen/meshes/sink/kitchen_only_parte_de_arriba_lavavajillas.obj"/>
             </geometry>
         </collision>
@@ -256,11 +256,11 @@
             <origin xyz="0.0 0.0 0.0" rpy="1.5714 0.0 0.0"/>
             <geometry>
-                <mesh filename="package://eut_urdf_models/meshes/sink/kitchen_only_cubiertos_lavavajillas.obj"/>
-            </geometry>
-        </visual>
-        <collision>
-            <origin xyz="0.0 0.0 0.0" rpy="1.5714 0.0 0.0"/>
-            <geometry>
-                <mesh filename="package://eut_urdf_models/meshes/sink/kitchen_only_cubiertos_lavavajillas.obj"/>
+                <mesh filename="package://sim_tiago_kitchen/meshes/sink/kitchen_only_cubiertos_lavavajillas.obj"/>
+            </geometry>
+        </visual>
+        <collision>
+            <origin xyz="0.0 0.0 0.0" rpy="1.5714 0.0 0.0"/>
+            <geometry>
+                <mesh filename="package://sim_tiago_kitchen/meshes/sink/kitchen_only_cubiertos_lavavajillas.obj"/>
             </geometry>
         </collision>
