Commit message: Fix FILTERING union map - CENTERING map_gen - NEW MAPS - change objects

File: tiago/tiago_robot/tiago_description/robots/tiago.urdf.xacro (robot description, xacro)
@@ -150,5 +150,5 @@
         </arm>
        <forces_angle_tolerance>100</forces_angle_tolerance>
-       <update_rate>100</update_rate>
+       <update_rate>500</update_rate>
        <grip_count_threshold>1</grip_count_threshold>
        <max_grip_count>2</max_grip_count>

File: tiago/tiago_robot/tiago_description/urdf/torso/torso.urdf.xacro (robot description, xacro)
@@ -149,4 +149,19 @@
     <xacro:torso_simple_transmission name="torso_lift" reduction="1.0" />
   </xacro:unless>
+  <joint name="${name}_footprint_joint" type="fixed">
+    <origin rpy="0 0 0" xyz="0.062 0 -0.888" />
+    <parent link="${name}_lift_link" />
+    <child link="${name}_footprint" />
+    <axis xyz="0 0 0" />
+  </joint>
+  <link name="${name}_footprint">
+    <inertial>
+      <origin rpy="0 0 0" xyz="0 0 0" />
+      <mass value="0.01" />
+      <inertia ixx="0.000001" ixy="0" ixz="0"
+               iyy="0.000001" iyz="0"
+               izz="0.000001" />
+    </inertial>
+  </link>
  </xacro:macro>
 </robot>
